Commit message: Add camera and lidar. Run Gazebo

File: description/camera.xacro (robot description, xacro)
@@ -1,6 +1,24 @@
 <?xml version="1.0"?>
 <robot xmlns:xacro="http://www.ros.org/wiki/xacro">
+    <!-- The next section shows an example of adding a sensor, in this case a depth camera. -->
+    <joint name="camera_joint" type="fixed">
+        <origin xyz="0.305 0 0.08" rpy="0 0 0"/>
+        <parent link="chassis"/>
+        <child link="camera_link"/>
+    </joint>
+    <link name="camera_link">
+        <visual>
+            <geometry>
+                <box size="0.010 0.03 0.03"/>
+            </geometry>
+            <material name="red"/>
+        </visual>
+    </link>
+    <!-- Due to a quirk of how cameras work, an extra joint/link is required to create an
+            "optical frame" for the sensor. That isn't the focus for this tutorial, but you can
+            look at https://www.ros.org/reps/rep-0103.html#suffix-frames for slightly more information. -->
+    <!-- First, create the link and joint for the optical frame -->
     <joint name="camera_optical_joint" type="fixed">
-        <origin xyz="0 0 0" rpy="-1.571 0 -1.571"/>
+        <origin xyz="0 0 0" rpy="${-pi/2} 0 ${-pi/2}"/>
         <parent link="camera_link"/>
         <child link="camera_link_optical"/>
@@ -8,17 +26,19 @@
     <link name="camera_link_optical"></link>
     <gazebo reference="camera_link">
-        <sensor type="camera" name="my_camera">
-            <update_rate>20</update_rate>
+        <material>Gazebo/Red</material>
+        <sensor type="camera" name="rgb_camera">
+            <pose> 0 0 0 0 0 0 </pose>
             <visualize>true</visualize>
-            <camera name="cam">
-                <horizontal_fov>1.3962634</horizontal_fov>
+            <update_rate>10</update_rate>
+            <camera>
+                <horizontal_fov>1.089</horizontal_fov>
                 <image>
+                    <format>R8B8G8</format>
                     <width>640</width>
                     <height>480</height>
-                    <format>R8B8G8</format>
                 </image>
                 <clip>
-                    <near>0.02</near>
-                    <far>300</far>
+                    <near>0.05</near>
+                    <far>8.0</far>
                 </clip>
                 <noise>
@@ -30,6 +50,4 @@
             <plugin name="camera_controller" filename="libgazebo_ros_camera.so">
                 <frame_name>camera_link_optical</frame_name>
-                <min_depth>0.1</min_depth>
-                <max_depth>500</max_depth>
             </plugin>
         </sensor>

File: description/robot.urdf.xacro (robot description, xacro)
@@ -3,3 +3,4 @@
     <xacro:include filename="robot_core.xacro"/>
     <xacro:include filename="gazebo_control.xacro"/>
+    <xacro:include filename="gazebo_lidar.xacro"/>
 </robot>

File: description/robot_core.xacro (robot description, xacro)
@@ -14,4 +14,7 @@
         <color rgba="0 0 0 1"/>
     </material>
+    <material name="red">
+        <color rgba="1 0 0 1"/>
+    </material>
     <!-- BASE LINK -->
     <link name="base_link">
@@ -19,7 +22,7 @@
     <!-- CHASSIS LINK -->
     <joint name="chassis_joint" type="fixed">
+        <origin xyz="-0.1 0 0"/>
         <parent link="base_link"/>
         <child link="chassis"/>
-        <origin xyz="-0.1 0 0"/>
     </joint>
     <link name="chassis">
@@ -123,3 +126,22 @@
         <mu2 value="0.001"/>
     </gazebo>
+    <gazebo>
+        <plugin name="gazebo_ros_joint_state_publisher"
+                filename="libgazebo_ros_joint_state_publisher.so">
+            <update_rate>20</update_rate>
+            <joint_name>left_wheel_joint</joint_name>
+            <joint_name>right_wheel_joint</joint_name>
+        </plugin>
+    </gazebo>
+    <!-- You'll probably want to add damping to the joints to stop them it flopping around.
+            e.g. <dynamics damping="10.0" friction="10.0"/> -->
+    <!-- Here's an example message to publish to test it:
+            ros2 topic pub -1 /set_joint_trajectory trajectory_msgs/msg/JointTrajectory  '{header: {frame_id: world}, joint_names: [slider_joint, arm_joint], points: [  {positions: {0.8,0.6}} ]}' -->
+    <gazebo>
+        <plugin name="gazebo_ros_joint_pose_trajectory" filename="libgazebo_ros_joint_pose_trajectory.so">
+            <update_rate>2</update_rate>
+            <dynamics damping="10.0" friction="10.0"/>
+        </plugin>
+    </gazebo>
+    <xacro:include filename="camera.xacro"/>
 </robot>
